File: hardware/cyberbrick-breakout/kicad/cyberbrick-breakout.kicad_pcb (KiCad board)
At the start: 2 copper layers, 85 x 70 mm, 33 parts

Commit message: Fix PCB: use fp_text for refs/values, correct KiCad 7 layer table, add UUIDs
Parts:
- removed ? (x4): , MountingHole:MountingHole_3.2mm_M3
- removed ? (x4): , Connector_JST:JST_SH_SM03B-SRSS-TB_1x03-1MP_P1.00mm_Horizontal
- removed ? (x4): , Capacitor_SMD:C_0402_1005Metric
- removed ? (x16): , Connector_JST:JST_SH_SM02B-SRSS-TB_1x02-1MP_P1.00mm_Horizontal
- removed ?: , Connector_PinHeader_2.54mm:PinHeader_2x09_P2.54mm_Vertical
- removed ?: , Connector_PinHeader_2.54mm:PinHeader_1x04_P2.54mm_Vertical
- removed ?: , Connector_PinHeader_2.54mm:PinHeader_1x02_P2.54mm_Vertical
- removed ? (x2): , Connector_PinSocket_2.54mm:PinSocket_1x08_P2.54mm_Vertical
- added C1: 100nF, Capacitor_SMD:C_0402_1005Metric, F.Cu at (10.0, 9.50)
- added C2: 100nF, Capacitor_SMD:C_0402_1005Metric, F.Cu at (23.0, 9.50)
- added C3: 100nF, Capacitor_SMD:C_0402_1005Metric, F.Cu at (36.0, 9.50)
- added C4: 100nF, Capacitor_SMD:C_0402_1005Metric, F.Cu at (49.0, 9.50)
- added H1: M3, MountingHole:MountingHole_3.2mm_M3, F.Cu at (3.50, 3.50)
- added H2: M3, MountingHole:MountingHole_3.2mm_M3, F.Cu at (81.5, 3.50)
- added H3: M3, MountingHole:MountingHole_3.2mm_M3, F.Cu at (3.50, 66.5)
- added H4: M3, MountingHole:MountingHole_3.2mm_M3, F.Cu at (81.5, 66.5)
- added J1: LX, Connector_JST:JST_SH_SM03B-SRSS-TB_1x03-1MP_P1.00mm_Horizontal, F.Cu at (10.0, 4.00)
- added J10: DL_LEFT, Connector_JST:JST_SH_SM02B-SRSS-TB_1x02-1MP_P1.00mm_Horizontal, F.Cu at (9.80, 62.0)
- added J11: DL_RIGHT, Connector_JST:JST_SH_SM02B-SRSS-TB_1x02-1MP_P1.00mm_Horizontal, F.Cu at (14.6, 62.0)
- added J12: DL_DOWN, Connector_JST:JST_SH_SM02B-SRSS-TB_1x02-1MP_P1.00mm_Horizontal, F.Cu at (19.4, 62.0)
- added J13: DR_UP, Connector_JST:JST_SH_SM02B-SRSS-TB_1x02-1MP_P1.00mm_Horizontal, F.Cu at (24.2, 62.0)
- added J14: DR_LEFT, Connector_JST:JST_SH_SM02B-SRSS-TB_1x02-1MP_P1.00mm_Horizontal, F.Cu at (29.0, 62.0)
- added J15: DR_RIGHT, Connector_JST:JST_SH_SM02B-SRSS-TB_1x02-1MP_P1.00mm_Horizontal, F.Cu at (33.8, 62.0)
- added J16: DR_DOWN, Connector_JST:JST_SH_SM02B-SRSS-TB_1x02-1MP_P1.00mm_Horizontal, F.Cu at (38.6, 62.0)
- added J17: SHL1, Connector_JST:JST_SH_SM02B-SRSS-TB_1x02-1MP_P1.00mm_Horizontal, F.Cu at (5.00, 66.5)
- added J18: SHL2, Connector_JST:JST_SH_SM02B-SRSS-TB_1x02-1MP_P1.00mm_Horizontal, F.Cu at (9.80, 66.5)
- added J19: SHR1, Connector_JST:JST_SH_SM02B-SRSS-TB_1x02-1MP_P1.00mm_Horizontal, F.Cu at (14.6, 66.5)
- added J2: LY, Connector_JST:JST_SH_SM03B-SRSS-TB_1x03-1MP_P1.00mm_Horizontal, F.Cu at (23.0, 4.00)
- added J20: SHR2, Connector_JST:JST_SH_SM02B-SRSS-TB_1x02-1MP_P1.00mm_Horizontal, F.Cu at (19.4, 66.5)
- added J21: START, Connector_JST:JST_SH_SM02B-SRSS-TB_1x02-1MP_P1.00mm_Horizontal, F.Cu at (24.2, 66.5)
- added J22: SELECT, Connector_JST:JST_SH_SM02B-SRSS-TB_1x02-1MP_P1.00mm_Horizontal, F.Cu at (29.0, 66.5)
- added J23: HOTKEY, Connector_JST:JST_SH_SM02B-SRSS-TB_1x02-1MP_P1.00mm_Horizontal, F.Cu at (33.8, 66.5)
- added J24: COIN, Connector_JST:JST_SH_SM02B-SRSS-TB_1x02-1MP_P1.00mm_Horizontal, F.Cu at (38.6, 66.5)
- added J3: RX, Connector_JST:JST_SH_SM03B-SRSS-TB_1x03-1MP_P1.00mm_Horizontal, F.Cu at (36.0, 4.00)
- added J4: RY, Connector_JST:JST_SH_SM03B-SRSS-TB_1x03-1MP_P1.00mm_Horizontal, F.Cu at (49.0, 4.00)
- added J6: MCP_BTNS, Connector_PinHeader_2.54mm:PinHeader_2x09_P2.54mm_Vertical, F.Cu at (76.5, 12.0)
- added J7: I2C, Connector_PinHeader_2.54mm:PinHeader_1x04_P2.54mm_Vertical, F.Cu at (76.5, 42.0)
- added J8: PWR_IN, Connector_PinHeader_2.54mm:PinHeader_1x02_P2.54mm_Vertical, F.Cu at (76.5, 56.0)
- added J9: DL_UP, Connector_JST:JST_SH_SM02B-SRSS-TB_1x02-1MP_P1.00mm_Horizontal, F.Cu at (5.00, 62.0)
- added U1A: ESP32-C3 top, Connector_PinSocket_2.54mm:PinSocket_1x08_P2.54mm_Vertical, F.Cu at (26.1, 17.4)
- added U1B: ESP32-C3 bot, Connector_PinSocket_2.54mm:PinSocket_1x08_P2.54mm_Vertical, F.Cu at (26.1, 32.6)
Other:
- board text added: "GPIO2=BOOT STRAP: no pulldown on J3!"
- board text added: "Verify U1 row spacing before ordering!"
- board text removed: "GPIO2=BOOT STRAP - no pulldown!"
