File: hardware/cyberbrick-breakout/kicad/cyberbrick-breakout.kicad_pcb (KiCad board)
At the start: 2 copper layers, 73 x 41 mm, 34 parts, among them J1 LX, J10 DL_LFT, J11 DL_RGT, J12 DL_DWN, J13 DR_UP, J14 DR_LFT, J15 DR_RGT, J16 DR_DWN, J17 SHL1, J18 SHL2, J19 SHR1, J2 LY, J20 SHR2, J21 START, J22 SEL, J23 HOTKEY, J24 COIN, J3 RX, J4 RY, J6A GPA, J6B GPB, J7 I2C, J8 PWR, J9 DL_UP, U1A ESP32-C3 top, U1B ESP32-C3 bot

Commit message: reviewed schematic
Parts:
- removed J6A: GPA, Connector_PinHeader_2.54mm:PinHeader_1x09_P2.54mm_Vertical
- removed J6B: GPB, Connector_PinHeader_2.54mm:PinHeader_1x09_P2.54mm_Vertical
- added C5: 100nF, Capacitor_SMD:C_0402_1005Metric, F.Cu at (148.5, 118.0)
- added MCP23017-E/SO: SOIC-28W_7.5x17.9mm_P1.27mm, Package_SO:SOIC-28W_7.5x17.9mm_P1.27mm, F.Cu at (151.0, 125.0)
- moved J7 29.1 mm to (142.5, 115.0), turned to 90 degrees
- moved J8 7.07 mm to (170.0, 112.0)
- moved U1B 0.44 mm to (118.0, 119.0)
Connections:
- J7 pad 3: VCC -> GND
- J7 pad 4: GND -> VCC
